File: yolouego.sch (KiCad schematic (older format))
At the start: 92 parts, among them J1 Conn_01x06, J2 Conn_01x02, J3 Conn_01x04, Q1 BSP129, Q2 Q_NMOS_GDS, Q3 MMBT3906, Q4 Q_PMOS_GDS, U1 REF5025AD, U14 MIC5219-3.3, U16 MIC5219-3.3, U2 OPA4376, U3 OPA4376, U4 NCP1117-5.0_SOT223, U5 NCP1117-5.0_SOT223, U8 STM32F373C8Tx, Y1 Crystal

Commit message: analog output
Parts:
- added C25, C26: C, stmbl-kicad-lib:C_0603, symbol device:C
- added J4: Conn_01x02, stmbl-kicad-lib:Pin_Header_Straight_1x02, symbol Connector:Conn_01x02
Connections:
- wire segments 300 -> 309
Changed lines of the file:
@@
 	1    0    0    -1
 $EndComp
-Wire Wire Line
-	4750 3300 4750 3500
-Wire Wire Line
-	4750 3700 4850 3700
-Connection ~ 4750 3500
-Wire Wire Line
-	4750 3500 4750 3700
-$Comp
-L power:GNDA #PWR0178
-U 1 1 5CAAD567
-P 4850 3700
-F 0 "#PWR0178" H 4850 3450 50  0001 C CNN
-F 1 "GNDA" H 4855 3527 50  0000 C CNN
-F 2 "" H 4850 3700 50  0001 C CNN
-F 3 "" H 4850 3700 50  0001 C CNN
-	1    4850 3700
-	1    0    0    -1
-$EndComp
-Connection ~ 4850 3700
-Wire Wire Line
-	4850 3700 4950 3700
 Text GLabel 10400 9900 0    50   Input ~ 0
 HEATER_HIGH
@@
 	10400 9900 10550 9900
 Connection ~ 10550 9900
+Text GLabel 4350 3300 0    50   Input ~ 0
+DAC3
+Wire Wire Line
+	4350 3300 4500 3300
+Wire Wire Line
+	5350 3400 5500 3400
+Wire Wire Line
+	5500 3400 5500 3900
+Wire Wire Line
+	5500 3900 4700 3900
+Wire Wire Line
+	4700 3900 4700 3500
+Wire Wire Line
+	4700 3500 4750 3500
+$Comp
+L device:C C25
+U 1 1 5CB1FEF6
+P 4500 3450
+F 0 "C25" H 4615 3496 50  0000 L CNN
+F 1 "C" H 4615 3405 50  0000 L CNN
+F 2 "stmbl-kicad-lib:C_0603" H 4538 3300 50  0001 C CNN
+F 3 "" H 4500 3450 50  0001 C CNN
+	1    4500 3450
+	1    0    0    -1
+$EndComp
+Connection ~ 4500 3300
+Wire Wire Line
+	4500 3300 4750 3300
+Wire Wire Line
+	4500 3600 4500 3700
+$Comp
+L power:GNDA #PWR0178
+U 1 1 5CB3C94B
+P 4500 3700
+F 0 "#PWR0178" H 4500 3450 50  0001 C CNN
+F 1 "GNDA" H 4505 3527 50  0000 C CNN
+F 2 "" H 4500 3700 50  0001 C CNN
+F 3 "" H 4500 3700 50  0001 C CNN
+	1    4500 3700
+	1    0    0    -1
+$EndComp
+$Comp
+L Connector:Conn_01x02 J4
+U 1 1 5CB3D4FD
+P 6050 3400
+F 0 "J4" H 6130 3392 50  0000 L CNN
+F 1 "Conn_01x02" H 6130 3301 50  0000 L CNN
+F 2 "stmbl-kicad-lib:Pin_Header_Straight_1x02" H 6050 3400 50  0001 C CNN
+F 3 "~" H 6050 3400 50  0001 C CNN
+	1    6050 3400
+	1    0    0    -1
+$EndComp
+$Comp
+L device:C C26
+U 1 1 5CB3E04D
+P 5700 3550
+F 0 "C26" H 5815 3596 50  0000 L CNN
+F 1 "C" H 5815 3505 50  0000 L CNN
+F 2 "stmbl-kicad-lib:C_0603" H 5738 3400 50  0001 C CNN
+F 3 "" H 5700 3550 50  0001 C CNN
+	1    5700 3550
+	1    0    0    -1
+$EndComp
+Connection ~ 5500 3400
+Wire Wire Line
+	5500 3400 5700 3400
+Connection ~ 5700 3400
+Wire Wire Line
+	5700 3400 5850 3400
+$Comp
+L power:GNDA #PWR0179
+U 1 1 5CB76983
+P 5700 3750
+F 0 "#PWR0179" H 5700 3500 50  0001 C CNN
+F 1 "GNDA" H 5705 3577 50  0000 C CNN
+F 2 "" H 5700 3750 50  0001 C CNN
+F 3 "" H 5700 3750 50  0001 C CNN
+	1    5700 3750
+	1    0    0    -1
+$EndComp
+Wire Wire Line
+	5700 3700 5700 3750
+Wire Wire Line
+	5850 3500 5850 3750
+Wire Wire Line
+	5850 3750 5700 3750
+Connection ~ 5700 3750
 $EndSCHEMATC

Commit message: kicad is best cad.... D:
Parts:
- removed U5: NCP1117-5.0_SOT223, TO_SOT_Packages_SMD:SOT-223-3_TabPin2, symbol regul:NCP1117-5.0_SOT223
- added U?: NCP1117-5.0_SOT223, TO_SOT_Packages_SMD:SOT-223-3_TabPin2, symbol Regulator_Linear:NCP1117-5.0_SOT223
- C1, C10, C11, C12, C13, C14, C16, C17, C18, C19, C2, C20, C21, C22, C23, C24, C25, C26, C3, C4, C5, C6, C7, C9: symbol device:C -> stmbl:C
- C15, C8: symbol device:CP -> stmbl:CP
- D1: symbol device:D -> stmbl:D
- J1: symbol Connector:Conn_01x06 -> stmbl:CONN_01X06
- J2, J4: symbol Connector:Conn_01x02 -> stmbl:CONN_01X02
- J3: symbol Connector:Conn_01x04 -> stmbl:CONN_01X04
- L1, L2, L3, L4: symbol device:Ferrite_Bead -> Device:Ferrite_Bead
- Q1: symbol Transistor:BSP129 -> Transistor_FET:BSP129
- Q2: symbol device:Q_NMOS_GDS -> Device:Q_NMOS_GDS
- Q3: symbol Transistor:MMBT3906 -> Transistor_BJT:MMBT3906
- Q4: symbol device:Q_PMOS_GDS -> Device:Q_PMOS_GDS
- R1, R10, R11, R12, R13, R14, R15, R16, R17, R18, R19, R20, R21, R22, R23, R24, R25, R26, R28, R30, R31, R32, R33, R34, R39, R41, R42, R6, R7, R9: symbol device:R -> stmbl:R
- U1: symbol references:REF5025AD -> Reference_Voltage:REF5025AD
- U14, U16: symbol regul:MIC5219-3.3 -> Regulator_Linear:MIC5219-3.3
- U2, U3: symbol linear:OPA4376 -> Amplifier_Operational:OPA4376
- U4: symbol regul:NCP1117-5.0_SOT223 -> Regulator_Linear:NCP1117-5.0_SOT223
- U8: symbol MCU_ST_STM32:STM32F373C8Tx -> MCU_ST_STM32F3:STM32F373CBTx
Connections:
- wire segments 309 -> 291
Other:
- moved on the sheet: JP1, Y1
