File: yolouego.sch (KiCad schematic (older format))
At the start: 101 parts, among them J1 Conn_01x06, J2 Conn_01x02, J3 Conn_01x04, J4 Conn_01x02, Q1 BSP129, Q2 Q_NMOS_GDS, Q3 MMBT3906, Q4 Q_PMOS_GDS, U1 REF5025AD, U14 MIC5219-3.3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

Commit message: add 3.3V on programming header
Parts:
- added J5: CONN_01X03, stmbl:Pin_Header_Straight_1x03, symbol stmbl:CONN_01X03
- added R2: R, stmbl-kicad-lib:R_0603, symbol stmbl:R
- added unit 5 of U2
- added unit 5 of U3
- added U5: MCP2558FD-xSN, Package_SO:SOIC-8_3.9x4.9mm_P1.27mm, symbol Interface_CAN_LIN:MCP2558FD-xSN
- J3: footprint stmbl-kicad-lib:Pin_Header_Straight_1x04 -> Connector_PinHeader_2.54mm:PinHeader_1x05_P2.54mm_Vertical; symbol stmbl:CONN_01X04 -> stmbl:CONN_01X05
- gave numbers to parts that had none: 1
Connections:
- net +3V3: now also J3.5 (Pin_5), U5.5 (VIO)
- net +5VA: now also U2.4 (V+), U3.4 (V+)
- net +5VD: now also U5.3 (VDD)
- net 2.5VrefA: now also U2.5 (+); no longer U2.3 (+)
- net DAC3: now also U2.12 (+); no longer U2.3 (+)
- net GNDA: now also U2.11 (V-), U3.11 (V-)
- net GNDD: now also J5.3 (Pin_3), U5.2 (VSS)
- net HEATER_CUR: now also U2.8; no longer U2.1
- net HTR_VOLT_HIGH: now also C9.1
- net HTR_VOLT_LOW: now also C4.1
- net PIN1: now also C14.2
- net PIN5: now also C14.1
- net PIN6: now also C11.1
- net VGND: now also U2.6 (-), U2.7; no longer U2.1, U2.2 (-)
- net at C13.1, Q4.2 (D), U4.3 (VI)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: now also C15.1, C8.1
- net at R42.2: now also C13.2, D4.1 (K)
- net at C10.1, R30.1: now also U2.10 (+); no longer U2.3 (+)
- net at R31.1, R34.2: now also U2.9 (-); no longer U2.2 (-)
- net at R12.1, R18.2: now also U3.10 (+); no longer U3.3 (+)
- net at R13.1, R20.2: now also U3.9 (-); no longer U3.2 (-)
- net at R23.1, R25.2: now also U3.8; no longer U3.1
- net at R14.1, R19.2: now also U3.12 (+); no longer U3.3 (+)
- net at R15.1, R21.2: now also U3.13 (-); no longer U3.2 (-)
- net at R24.1, R26.1: now also U3.14; no longer U3.1
- net at R35.1, R37.2: now also U3.5 (+); no longer U3.3 (+)
- net at R36.1, R38.2: now also U3.6 (-); no longer U3.2 (-)
- net at R38.1, R40.2: now also U3.7; no longer U3.1
- net TX: now reaches U8.30 (PA9)
- net RX: now reaches U8.31 (PA10)
- net at U8.32 (PA11): now also U5.4 (RXD)
- net at U8.33 (PA12): now also U5.1 (TXD)
- net at U8.38 (PA15): now also U5.8 (S)
- net at C26.1, J4.1 (Pin_1): now also U2.13 (-), U2.14; no longer U2.1, U2.2 (-)
- new net: J5.2 (Pin_2), R2.2, U5.6 (CANL)
- new net: J5.1 (Pin_1), R2.1, U5.7 (CANH)
Other:
- moved on the sheet: R18, R19, R23, R24

Commit message: fix sot23
Parts:
- Q1: symbol Transistor_FET:BSP129 -> stmbl:NFET
- U14, U16: symbol Regulator_Linear:MIC5219-3.3 -> Regulator_Linear:MIC5219-3.3YM5
Connections:
- net GNDPWR: now also Q1.2 (S); no longer Q1.3 (S)
- net at Q2.1 (G), R22.1: now also Q1.3 (D); no longer Q1.2 (D)
Other:
- moved on the sheet: Q1
Changed lines of the file:
@@
 $EndComp
 $Comp
-L Regulator_Linear:MIC5219-3.3 U16
+L Regulator_Linear:MIC5219-3.3YM5 U16
 U 1 1 5A70AB53
 P 14050 1000
@@
 	11300 2550 11300 2600
 $Comp
-L Regulator_Linear:MIC5219-3.3 U14
+L Regulator_Linear:MIC5219-3.3YM5 U14
 U 1 1 5A71359B
 P 13000 1900
@@
 $EndComp
 $Comp
-L Transistor_FET:BSP129 Q1
+L stmbl:NFET Q1
 U 1 1 5A7227E6
-P 6300 10550
-F 0 "Q1" H 6505 10596 50  0000 L CNN
-F 1 "BSP129" H 6505 10505 50  0000 L CNN
-F 2 "stmbl-kicad-lib:SOT-23" H 6500 10475 50  0001 L CIN
-F 3 "https://www.infineon.com/dgdl/Infineon-BSP129-DS-v01_42-en.pdf?fileId=db3a30433c1a8752013c1fc296d2395f" H 6300 10550 50  0001 L CNN
-	1    6300 10550
+P 6350 10500
+F 0 "Q1" H 6555 10546 50  0000 L CNN
+F 1 "BSP129" H 6555 10455 50  0000 L CNN
+F 2 "stmbl-kicad-lib:SOT-23" H 6550 10425 50  0001 L CIN
+F 3 "https://www.infineon.com/dgdl/Infineon-BSP129-DS-v01_42-en.pdf?fileId=db3a30433c1a8752013c1fc296d2395f" H 6350 10500 50  0001 L CNN
+	1    6350 10500
 	1    0    0    -1
 $EndComp
@@
 Connection ~ 6400 10200
 Wire Wire Line
-	6400 10200 6400 10350
+	6400 10200 6400 10300
 Wire Wire Line
 	6400 9750 6400 9850
@@
 	1    0    0    -1
 $EndComp
-Wire Wire Line
-	6400 10750 6400 10800
 Wire Wire Line
 	7150 10800 7150 10850
@@
 Wire Wire Line
 	8700 6800 8700 6900
+Wire Wire Line
+	6400 10700 6400 10800
 $EndSCHEMATC
