File: yolouego.kicad_pcb (KiCad board)
At the start: 4 copper layers, 50 x 50 mm, 92 parts, among them J1 Conn_01x06, J2 Conn_01x02, J3 Conn_01x04, Q1 BSP129, Q2 Q_NMOS_GDS, Q3 MMBT3906, Q4 Q_PMOS_GDS, U1 REF5025AD, U14 MIC5219-3.3, U16 MIC5219-3.3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

Commit message: analog output
Parts:
- added C25: C, stmbl-kicad-lib:C_0603, F.Cu at (119.0, 78.6)
- added C26: C, stmbl-kicad-lib:C_0603, F.Cu at (123.4, 72.2)
- added J4: Conn_01x02, stmbl-kicad-lib:Pin_Header_Straight_1x02, F.Cu at (119.0, 70.6)
- moved L4 0.80 mm to (114.6, 67.6)
Connections:
- U2 pad 12: GNDA -> DAC3
- U2 pad 13: GNDA -> Net-(C26-Pad1)
- U2 pad 14: Net-(U2-Pad14) -> Net-(C26-Pad1)
Routing:
- net DAC3: track 0.00 -> 13.9 mm, vias 0 -> 2
- net Net-(C26-Pad1): track 0.00 -> 11.5 mm
- net NRST: track 25.8 -> 23.7 mm
- net GNDA: vias 15 -> 18

Commit message: add 3.3V on programming header
Parts:
- added J5: CONN_01X03, stmbl:Pin_Header_Straight_1x03, F.Cu at (97.0, 70.6)
- added U5: MCP2558FD-xSN, Package_SO:SOIC-8_3.9x4.9mm_P1.27mm, F.Cu at (101.5, 73.7)
- J3: footprint stmbl-kicad-lib:Pin_Header_Straight_1x04 -> Connector_PinHeader_2.54mm:PinHeader_1x05_P2.54mm_Vertical
- moved C8 6.94 mm to (92.8, 72.4), turned to 90 degrees
- moved U5 2.01 mm to (98.4, 64.5)
- moved J3 1.98 mm to (111.5, 69.2)
- moved C3 0.10 mm to (131.8, 93.7)
Connections:
- net Net-(U8-Pad30) renamed TX
- net Net-(U8-Pad31) renamed RX
Routing:
- net +5VA: track 55.8 -> 13.0 mm, vias 2 -> 5
- net Net-(U5-Pad1): track 0.00 -> 24.3 mm, vias 0 -> 2
- net Net-(U5-Pad8): track 0.00 -> 24.1 mm, vias 0 -> 2
- net Net-(U5-Pad4): track 0.00 -> 20.5 mm, vias 0 -> 2
- net +5VD: track 28.9 -> 36.8 mm
- net Net-(J5-Pad2): track 0.00 -> 6.59 mm
- net Net-(J5-Pad1): track 0.00 -> 5.49 mm
- net Net-(C13-Pad1): track 59.7 -> 63.9 mm
- net GNDPWR: track 44.9 -> 48.8 mm
- net NRST: track 23.7 -> 26.7 mm
- net Net-(Q2-Pad3): track 36.1 -> 38.7 mm
- net +3V3: track 23.8 -> 25.8 mm, vias 7 -> 8
- net Net-(J3-Pad2): track 9.40 -> 11.3 mm
- net Net-(J3-Pad4): track 4.08 -> 6.02 mm
- net +3.3VA: track 35.9 -> 37.5 mm
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- added copper zone on In2.Cu, net +5VA
- added copper zone on B.Cu, net GNDPWR
Other:
- rule trace_min: 0.2 -> 0.15
