File: yolouego.kicad_pcb (KiCad board)
At the start: 4 copper layers, 50 x 50 mm, 97 parts, among them J1 Conn_01x06, J2 Conn_01x02, J3 Conn_01x04, J4 Conn_01x02, J5 CONN_01X03, Q1 BSP129, Q2 Q_NMOS_GDS, Q3 MMBT3906, Q4 Q_PMOS_GDS, U1 REF5025AD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

Commit message: fix sot23
Parts:
- removed the U5 at (98.4, 64.5)
- added R2: R, stmbl-kicad-lib:R_0603, F.Cu at (101.4, 68.8)
- added U6: NCP1117-5.0_SOT223, TO_SOT_Packages_SMD:SOT-223-3_TabPin2, F.Cu at (98.4, 64.4)
- turned Q1 to 270 degrees
Connections:
- Q1 pad 2: Net-(Q1-Pad2) -> GNDPWR
- Q1 pad 3: GNDPWR -> Net-(Q1-Pad3)
- Q2 pad 1: Net-(Q1-Pad2) -> Net-(Q1-Pad3)
- R22 pad 1: Net-(Q1-Pad2) -> Net-(Q1-Pad3)
Routing:
- net Net-(Q1-Pad2): track 9.30 -> 0.00 mm
- net Net-(Q1-Pad3): track 0.00 -> 8.78 mm
- net Net-(Q1-Pad1): track 5.21 -> 2.90 mm
- net Net-(J5-Pad1): track 5.49 -> 7.78 mm
- net Net-(J5-Pad2): track 6.59 -> 8.80 mm
- net Net-(C13-Pad1): track 63.9 -> 62.9 mm
- net GNDD: vias 18 -> 17
- net +5VA: vias 5 -> 31
- added copper zone on F.Cu, net +5VA
